File: sim_work/electrometer_362.kicad_sch (KiCad schematic)
At the start: 8 parts, among them U1 ADA4530-1

Commit message: Fix schematic connections, add docs and repo portability
- Input filters: R rotation=90 (horizontal), ESD diode rotations fixed,
  junction dots at cathode-signal connection, wires to GND symbols
- Relay ladder: flyback diode rotation 270->90 (K top, A bottom)
- Electrometer/Mux TIA: 4 junction dots each at T-junctions
- AD636 RMS detector: proper IC box with pin labels replaces text-only
- Oscillator blocks: D_Zener symbol, L-shaped cathode routing
- TIA blocks: title/function annotations on all 5 blocks
- New: requirements.txt, docs/oscillator_guide.md
- D_Zener.kicad_sym added to bundled symbols/
- .gitignore updated for docs/ and requirements.txt
- README updated with pip install -r requirements.txt
- PROJECT.md session 9 changelog
- SimGUI builds clean (0 errors)

Co-Authored-By: Claude Opus 4.6 <noreply@anthropic.com>
Connections:
- net AIN1: now also R3.2, R4.1
- net TRIAX_IN: now also R1.1
Other:
- note added: "ADA4530-1 TIA, 4-range relay-switched Rf (10M-10G), 24-bit ADC"
- note added: "ADC reads differential (TIA_OUT - VREF). Single 3.3V supply."
- note added: "ELECTROMETER TIA (ADuCM362 PLATFORM)"
- note added: "FUNCTION: Complete electrometer front-end. TIA converts current to"
- note added: "voltage. Relay ladder selects range. ADuCM362 24-bit sigma-delta"
Changed lines of the file:
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@@
 		(instances
 			(project "Electrometer TIA - ADuCM362"
-				(path "/f7fbb0e7-8495-472f-9e82-ab7e8e519fa6"
+				(path "/2a7435c9-0942-493c-8e3c-deaa9490a333"
 					(reference "U1")
 					(unit 1)
@@
 		(instances
 			(project "Electrometer TIA - ADuCM362"
-				(path "/f7fbb0e7-8495-472f-9e82-ab7e8e519fa6"
+				(path "/2a7435c9-0942-493c-8e3c-deaa9490a333"
 					(reference "R1")
 					(unit 1)
@@
 		(instances
 			(project "Electrometer TIA - ADuCM362"
-				(path "/f7fbb0e7-8495-472f-9e82-ab7e8e519fa6"
+				(path "/2a7435c9-0942-493c-8e3c-deaa9490a333"
 					(reference "C1")
 					(unit 1)
@@
 		(instances
 			(project "Electrometer TIA - ADuCM362"
-				(path "/f7fbb0e7-8495-472f-9e82-ab7e8e519fa6"
+				(path "/2a7435c9-0942-493c-8e3c-deaa9490a333"
 					(reference "R3")
 					(unit 1)
@@
 		(instances
 			(project "Electrometer TIA - ADuCM362"
-				(path "/f7fbb0e7-8495-472f-9e82-ab7e8e519fa6"
+				(path "/2a7435c9-0942-493c-8e3c-deaa9490a333"
 					(reference "R4")
 					(unit 1)
@@
 		(instances
 			(project "Electrometer TIA - ADuCM362"
-				(path "/f7fbb0e7-8495-472f-9e82-ab7e8e519fa6"
+				(path "/2a7435c9-0942-493c-8e3c-deaa9490a333"
 					(reference "C2")
 					(unit 1)
@@
 		(instances
 			(project "Electrometer TIA - ADuCM362"
-				(path "/f7fbb0e7-8495-472f-9e82-ab7e8e519fa6"
+				(path "/2a7435c9-0942-493c-8e3c-deaa9490a333"
 					(reference "R2")
 					(unit 1)
@@
 		(instances
 			(project "Electrometer TIA - ADuCM362"
-				(path "/f7fbb0e7-8495-472f-9e82-ab7e8e519fa6"
+				(path "/2a7435c9-0942-493c-8e3c-deaa9490a333"
 					(reference "#PWR01")
 					(unit 1)
@@
 		(instances
 			(project "Electrometer TIA - ADuCM362"
-				(path "/f7fbb0e7-8495-472f-9e82-ab7e8e519fa6"
+				(path "/2a7435c9-0942-493c-8e3c-deaa9490a333"
 					(reference "#PWR02")
 					(unit 1)
@@
 		(instances
 			(project "Electrometer TIA - ADuCM362"
-				(path "/f7fbb0e7-8495-472f-9e82-ab7e8e519fa6"
+				(path "/2a7435c9-0942-493c-8e3c-deaa9490a333"
 					(reference "#PWR03")
 					(unit 1)
@@
 		(instances
 			(project "Electrometer TIA - ADuCM362"
-				(path "/f7fbb0e7-8495-472f-9e82-ab7e8e519fa6"
+				(path "/2a7435c9-0942-493c-8e3c-deaa9490a333"
 					(reference "#PWR04")
 					(unit 1)
@@
 		(instances
 			(project "Electrometer TIA - ADuCM362"
-				(path "/f7fbb0e7-8495-472f-9e82-ab7e8e519fa6"
+				(path "/2a7435c9-0942-493c-8e3c-deaa9490a333"
 					(reference "#PWR05")
 					(unit 1)
@@
 		(instances
 			(project "Electrometer TIA - ADuCM362"
-				(path "/f7fbb0e7-8495-472f-9e82-ab7e8e519fa6"
+				(path "/2a7435c9-0942-493c-8e3c-deaa9490a333"
 					(reference "#PWR06")
 					(unit 1)
@@
 		(instances
 			(project "Electrometer TIA - ADuCM362"
-				(path "/f7fbb0e7-8495-472f-9e82-ab7e8e519fa6"
+				(path "/2a7435c9-0942-493c-8e3c-deaa9490a333"
 					(reference "V1")
 					(unit 1)
@@
 		(instances
 			(project "Electrometer TIA - ADuCM362"
-				(path "/f7fbb0e7-8495-472f-9e82-ab7e8e519fa6"
+				(path "/2a7435c9-0942-493c-8e3c-deaa9490a333"
 					(reference "#PWR07")
 					(unit 1)
@@
 			(type default)
 		)
+	)
+	(junction
+		(at 96.52 109.22)
+		(diameter 0)
+		(color 0 0 0 0)
+	)
+	(junction
+		(at 96.52 96.52)
+		(diameter 0)
+		(color 0 0 0 0)
+	)
+	(junction
+		(at 124.46 96.52)
+		(diameter 0)
+		(color 0 0 0 0)
+	)
+	(junction
+		(at 78.74 114.3)
+		(diameter 0)
+		(color 0 0 0 0)
 	)
 	(label "AIN0"
@@
 		)
 	)
+	(text "ELECTROMETER TIA (ADuCM362 PLATFORM)"
+		(exclude_from_sim no)
+		(at 20.32 15.24 0.0000)
+		(effects
+			(font
+				(size 4 4)
+				(bold yes)
+			)
+			(justify left)
+		)
+	)
+	(text "ADA4530-1 TIA, 4-range relay-switched Rf (10M-10G), 24-bit ADC"
+		(exclude_from_sim no)
+		(at 20.32 30.48 0.0000)
+		(effects
+			(font
+				(size 2.5 2.5)
+			)
+			(justify left)
+		)
+	)
+	(text "FUNCTION: Complete electrometer front-end. TIA converts current to"
+		(exclude_from_sim no)
+		(at 20.32 43.18 0.0000)
+		(effects
+			(font
+				(size 1.8 1.8)
+			)
+			(justify left)
+		)
+	)
+	(text "voltage. Relay ladder selects range. ADuCM362 24-bit sigma-delta"
+		(exclude_from_sim no)
+		(at 20.32 53.34 0.0000)
+		(effects
+			(font
+				(size 1.8 1.8)
+			)
+			(justify left)
+		)
+	)
+	(text "ADC reads differential (TIA_OUT - VREF). Single 3.3V supply."
+		(exclude_from_sim no)
+		(at 20.32 63.5 0.0000)
+		(effects
+			(font
+				(size 1.8 1.8)
+			)
+			(justify left)
+		)
+	)

Commit message: Add comparison mode, fix SimGUI subprocess popups, DAC7800 IC boxes
- SimGUI: fix Python path detection (FindPython searches Python312/313/311)
- SimGUI: suppress console popup windows (CREATE_NO_WINDOW for subprocess)
- SimGUI: add Comparison project (MDAC vs Analog oscillator side-by-side)
- SimGUI: fix async wrapping (direct await instead of Task.Run)
- Pipeline: draw DAC7800 as proper IC box with pin labels (VREF/IOUT/VCTRL)
- Pipeline: fix electrometer_362 layout (spacing, junction dots at T-junctions)
- Pipeline: fix summing amp gain annotations (BP=-0.455, not -2.2)
- Pipeline: add analog_osc command for friend's SVF oscillator simulation
- Docs: comparison_guide.md, updated README and PROJECT tracker

Co-Authored-By: Claude Opus 4.6 <noreply@anthropic.com>
Connections:
- net +3.3V: now also U1.4 (V-); no longer U1.7 (V+)
- net AIN1: now also C2.1, U1.2 (-); no longer U1.3 (+)
- net GND: now also U1.7 (V+); no longer U1.4 (V-)
- net TRIAX_IN: now also U1.3 (+); no longer U1.2 (-)
Changed lines of the file:
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@@
 		(lib_id "LM741:LM741")
 		(at 116.84 111.76 0)
-		(mirror x)
 		(unit 1)
 		(exclude_from_sim no)
@@
 		(instances
 			(project "Electrometer TIA - ADuCM362"
-				(path "/301a4b19-4aea-4be6-b0e1-3df22b423670"
+				(path "/24bf9fde-d8d7-47e7-9f50-dfc7fc70fb36"
 					(reference "U1")
 					(unit 1)
@@
 	(symbol
 		(lib_id "R:R")
-		(at 116.84 96.52 90)
+		(at 116.84 86.36 90)
 		(unit 1)
 		(exclude_from_sim no)
@@
 		(fields_autoplaced no)
 		(property "Reference" "R1"
-			(at 116.84 98.552 180)
+			(at 116.84 88.392 180)
 			(effects
 				(font
@@
 		)
 		(property "Value" "1G"
-			(at 116.84 96.52 180)
+			(at 116.84 86.36 180)
 			(effects
 				(font
@@
 		(instances
 			(project "Electrometer TIA - ADuCM362"
-				(path "/301a4b19-4aea-4be6-b0e1-3df22b423670"
+				(path "/24bf9fde-d8d7-47e7-9f50-dfc7fc70fb36"
 					(reference "R1")
 					(unit 1)
@@
 	(symbol
 		(lib_id "C:C")
-		(at 116.84 88.9 90)
+		(at 116.84 76.2 90)
 		(unit 1)
 		(exclude_from_sim no)
@@
 		(fields_autoplaced no)
 		(property "Reference" "C1"
-			(at 114.3 89.535 90)
+			(at 114.3 76.835 90)
 			(effects
 				(font
@@
 		)
 		(property "Value" "10pF"
-			(at 119.38 89.535 90)
+			(at 119.38 76.835 90)
 			(effects
 				(font
@@
 		(instances
 			(project "Electrometer TIA - ADuCM362"
-				(path "/301a4b19-4aea-4be6-b0e1-3df22b423670"
+				(path "/24bf9fde-d8d7-47e7-9f50-dfc7fc70fb36"
 					(reference "C1")
 					(unit 1)
@@
 		(instances
 			(project "Electrometer TIA - ADuCM362"
-				(path "/301a4b19-4aea-4be6-b0e1-3df22b423670"
+				(path "/24bf9fde-d8d7-47e7-9f50-dfc7fc70fb36"
 					(reference "R3")
 					(unit 1)
@@
 		(instances
 			(project "Electrometer TIA - ADuCM362"
-				(path "/301a4b19-4aea-4be6-b0e1-3df22b423670"
+				(path "/24bf9fde-d8d7-47e7-9f50-dfc7fc70fb36"
 					(reference "R4")
 					(unit 1)
@@
 		(instances
 			(project "Electrometer TIA - ADuCM362"
-				(path "/301a4b19-4aea-4be6-b0e1-3df22b423670"
+				(path "/24bf9fde-d8d7-47e7-9f50-dfc7fc70fb36"
 					(reference "C2")
 					(unit 1)
@@
 		(instances
 			(project "Electrometer TIA - ADuCM362"
-				(path "/301a4b19-4aea-4be6-b0e1-3df22b423670"
+				(path "/24bf9fde-d8d7-47e7-9f50-dfc7fc70fb36"
 					(reference "R2")
 					(unit 1)
@@
 		(instances
 			(project "Electrometer TIA - ADuCM362"
-				(path "/301a4b19-4aea-4be6-b0e1-3df22b423670"
+				(path "/24bf9fde-d8d7-47e7-9f50-dfc7fc70fb36"
 					(reference "#PWR01")
 					(unit 1)
@@
 		(instances
 			(project "Electrometer TIA - ADuCM362"
-				(path "/301a4b19-4aea-4be6-b0e1-3df22b423670"
+				(path "/24bf9fde-d8d7-47e7-9f50-dfc7fc70fb36"
 					(reference "#PWR02")
 					(unit 1)
@@
 		(instances
 			(project "Electrometer TIA - ADuCM362"
-				(path "/301a4b19-4aea-4be6-b0e1-3df22b423670"
+				(path "/24bf9fde-d8d7-47e7-9f50-dfc7fc70fb36"
 					(reference "#PWR03")
 					(unit 1)
@@
 		(instances
 			(project "Electrometer TIA - ADuCM362"
-				(path "/301a4b19-4aea-4be6-b0e1-3df22b423670"
+				(path "/24bf9fde-d8d7-47e7-9f50-dfc7fc70fb36"
 					(reference "#PWR04")
 					(unit 1)
@@
 		(instances
 			(project "Electrometer TIA - ADuCM362"
-				(path "/301a4b19-4aea-4be6-b0e1-3df22b423670"
+				(path "/24bf9fde-d8d7-47e7-9f50-dfc7fc70fb36"
 					(reference "#PWR05")
 					(unit 1)
@@
 		(instances
 			(project "Electrometer TIA - ADuCM362"
-				(path "/301a4b19-4aea-4be6-b0e1-3df22b423670"
+				(path "/24bf9fde-d8d7-47e7-9f50-dfc7fc70fb36"
 					(reference "#PWR06")
 					(unit 1)
@@
 		(instances
 			(project "Electrometer TIA - ADuCM362"
-				(path "/301a4b19-4aea-4be6-b0e1-3df22b423670"
+				(path "/24bf9fde-d8d7-47e7-9f50-dfc7fc70fb36"
 					(reference "V1")
 					(unit 1)
@@
 		(instances
 			(project "Electrometer TIA - ADuCM362"
-				(path "/301a4b19-4aea-4be6-b0e1-3df22b423670"
+				(path "/24bf9fde-d8d7-47e7-9f50-dfc7fc70fb36"
 					(reference "#PWR07")
 					(unit 1)
@@
 	(wire
 		(pts
-			(xy 96.52 96.52) (xy 113.03 96.52)
-		)
-		(stroke
-			(width 0)
-			(type default)
-		)
-	)
-	(wire
-		(pts
-			(xy 120.65 96.52) (xy 124.46 96.52)
-		)
-		(stroke
-			(width 0)
-			(type default)
-		)
-	)
-	(wire
-		(pts
-			(xy 124.46 96.52) (xy 124.46 111.76)
-		)
-		(stroke
-			(width 0)
-			(type default)
-		)
-	)
-	(wire
-		(pts
-			(xy 96.52 88.9) (xy 113.03 88.9)
-		)
-		(stroke
-			(width 0)
-			(type default)
-		)
-	)
-	(wire
-		(pts
-			(xy 120.65 88.9) (xy 124.46 88.9)
-		)
-		(stroke
-			(width 0)
-			(type default)
-		)
-	)
-	(wire
-		(pts
-			(xy 124.46 88.9) (xy 124.46 96.52)
+			(xy 96.52 86.36) (xy 113.03 86.36)
+		)
+		(stroke
+			(width 0)
+			(type default)
+		)
+	)
+	(wire
+		(pts
+			(xy 120.65 86.36) (xy 124.46 86.36)
+		)
+		(stroke
+			(width 0)
+			(type default)
+		)
+	)
+	(wire
+		(pts
+			(xy 124.46 86.36) (xy 124.46 111.76)
+		)
+		(stroke
+			(width 0)
+			(type default)
+		)
+	)
+	(wire
+		(pts
+			(xy 96.52 76.2) (xy 113.03 76.2)
+		)
+		(stroke
+			(width 0)
+			(type default)
+		)
+	)
+	(wire
+		(pts
+			(xy 120.65 76.2) (xy 124.46 76.2)
+		)
+		(stroke
+			(width 0)
+			(type default)
+		)
+	)
+	(wire
+		(pts
+			(xy 124.46 76.2) (xy 124.46 86.36)
 		)
 		(stroke
@@
 	(wire
 		(pts
-			(xy 63.5 81.28) (xy 63.5 109.22)
-		)
-		(stroke
-			(width 0)
-			(type default)
-		)
-	)
-	(wire
-		(pts
-			(xy 63.5 81.28) (xy 96.52 81.28)
-		)
-		(stroke
-			(width 0)
-			(type default)
-		)
-	)
-	(wire
-		(pts
-			(xy 96.52 81.28) (xy 96.52 109.22)
+			(xy 63.5 68.58) (xy 63.5 109.22)
+		)
+		(stroke
+			(width 0)
+			(type default)
+		)
+	)
+	(wire
+		(pts
+			(xy 63.5 68.58) (xy 96.52 68.58)
+		)
+		(stroke
+			(width 0)
+			(type default)
+		)
+	)
+	(wire
+		(pts
+			(xy 96.52 68.58) (xy 96.52 109.22)
 		)
 		(stroke
@@
 	)
 	(junction
-		(at 96.52 96.52)
+		(at 96.52 86.36)
 		(diameter 0)
 		(color 0 0 0 0)
 	)
 	(junction
-		(at 124.46 96.52)
+		(at 124.46 86.36)
 		(diameter 0)
 		(color 0 0 0 0)
 	)
 	(junction
+		(at 124.46 111.76)
+		(diameter 0)
+		(color 0 0 0 0)
+	)
+	(junction
 		(at 78.74 114.3)
+		(diameter 0)
+		(color 0 0 0 0)
+	)
+	(junction
+		(at 91.44 114.3)
 		(diameter 0)
 		(color 0 0 0 0)
@@
 	)
 	(label "TRIAX_IN"
-		(at 71.12 81.28 0)
+		(at 71.12 68.58 0)
 		(effects
 			(font
