File: sim_work/full_system.kicad_sch (KiCad schematic)
At the start: 114 parts, among them J1 INPUT_32PIN, J2 RTD_4WIRE, Q1 2N3904, Q2 2N3904, Q3 2N3904, Q4 2N3904, SW1 K1, SW2 K2, SW3 K3, SW4 K4, U1 MAX338, U2 MAX338, U3 ADA4530-1

Commit message: Add comparison mode, fix SimGUI subprocess popups, DAC7800 IC boxes
- SimGUI: fix Python path detection (FindPython searches Python312/313/311)
- SimGUI: suppress console popup windows (CREATE_NO_WINDOW for subprocess)
- SimGUI: add Comparison project (MDAC vs Analog oscillator side-by-side)
- SimGUI: fix async wrapping (direct await instead of Task.Run)
- Pipeline: draw DAC7800 as proper IC box with pin labels (VREF/IOUT/VCTRL)
- Pipeline: fix electrometer_362 layout (spacing, junction dots at T-junctions)
- Pipeline: fix summing amp gain annotations (BP=-0.455, not -2.2)
- Pipeline: add analog_osc command for friend's SVF oscillator simulation
- Docs: comparison_guide.md, updated README and PROJECT tracker

Co-Authored-By: Claude Opus 4.6 <noreply@anthropic.com>
Connections:
- net AIN1: now also U3.2 (-); no longer U3.3 (+)
- net CH_IN_1: now also D2.2 (A); no longer D2.1 (K)
- net CH_IN_10: now also D20.2 (A); no longer D20.1 (K)
- net CH_IN_11: now also D22.2 (A); no longer D22.1 (K)
- net CH_IN_12: now also D24.2 (A); no longer D24.1 (K)
- net CH_IN_13: now also D26.2 (A); no longer D26.1 (K)
- net CH_IN_14: now also D28.2 (A); no longer D28.1 (K)
- net CH_IN_15: now also D30.2 (A); no longer D30.1 (K)
- net CH_IN_16: now also D32.2 (A); no longer D32.1 (K)
- net CH_IN_2: now also D4.2 (A); no longer D4.1 (K)
- net CH_IN_3: now also D6.2 (A); no longer D6.1 (K)
- net CH_IN_4: now also D8.2 (A); no longer D8.1 (K)
- net CH_IN_5: now also D10.2 (A); no longer D10.1 (K)
- net CH_IN_6: now also D12.2 (A); no longer D12.1 (K)
- net CH_IN_7: now also D14.2 (A); no longer D14.1 (K)
- net CH_IN_8: now also D16.2 (A); no longer D16.1 (K)
- net CH_IN_9: now also D18.2 (A); no longer D18.1 (K)
- net GND: now also U3.7 (V+); no longer D1.2 (A), D10.2 (A), D11.2 (A), D12.2 (A), D13.2 (A), D14.2 (A), D15.2 (A), D16.2 (A), D17.2 (A), D18.2 (A), D19.2 (A), D2.2 (A), D20.2 (A), D21.2 (A), D22.2 (A), D23.2 (A), D24.2 (A), D25.2 (A), D26.2 (A), D27.2 (A), D28.2 (A), D29.2 (A), D3.2 (A), D30.2 (A), D31.2 (A), D32.2 (A), D4.2 (A), D5.2 (A), D6.2 (A), D7.2 (A), D8.2 (A), D9.2 (A), U3.4 (V-)
- net INV: now also U3.3 (+); no longer U3.2 (-)
- net VCC: now also U3.4 (V-); no longer U3.7 (V+)
- new net: D31.2 (A), D32.1 (K)
- new net: D29.2 (A), D30.1 (K)
- new net: D27.2 (A), D28.1 (K)
- new net: D21.2 (A), D22.1 (K)
- new net: D3.2 (A), D4.1 (K)
- new net: D5.2 (A), D6.1 (K)
- new net: D7.2 (A), D8.1 (K)
- new net: D1.2 (A), D2.1 (K)
- new net: D11.2 (A), D12.1 (K)
- new net: D23.2 (A), D24.1 (K)
- new net: D17.2 (A), D18.1 (K)
- new net: D25.2 (A), D26.1 (K)
- new net: D10.1 (K), D9.2 (A)
- new net: D15.2 (A), D16.1 (K)
- new net: D19.2 (A), D20.1 (K)
- new net: D13.2 (A), D14.1 (K)
