File: sim_work/inv_amp.kicad_sch (KiCad schematic)
At the start: 7 parts, among them U1 LM741

Commit message: Add comparison mode, fix SimGUI subprocess popups, DAC7800 IC boxes
- SimGUI: fix Python path detection (FindPython searches Python312/313/311)
- SimGUI: suppress console popup windows (CREATE_NO_WINDOW for subprocess)
- SimGUI: add Comparison project (MDAC vs Analog oscillator side-by-side)
- SimGUI: fix async wrapping (direct await instead of Task.Run)
- Pipeline: draw DAC7800 as proper IC box with pin labels (VREF/IOUT/VCTRL)
- Pipeline: fix electrometer_362 layout (spacing, junction dots at T-junctions)
- Pipeline: fix summing amp gain annotations (BP=-0.455, not -2.2)
- Pipeline: add analog_osc command for friend's SVF oscillator simulation
- Docs: comparison_guide.md, updated README and PROJECT tracker

Co-Authored-By: Claude Opus 4.6 <noreply@anthropic.com>
Connections:
- net +12V: now also U1.4 (V-); no longer U1.7 (V+)
- net -12V: now also U1.7 (V+); no longer U1.4 (V-)
- net GND: now also U1.2 (-); no longer U1.3 (+)
- net at R1.2: now also U1.3 (+); no longer U1.2 (-)
Changed lines of the file:
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@@
 		(lib_id "LM741:LM741")
 		(at 147.32 101.6 0)
-		(mirror x)
 		(unit 1)
 		(exclude_from_sim no)
@@
 		(instances
 			(project "Inverting Amplifier"
-				(path "/08241a88-1f4f-4518-809a-7c34a0316343"
+				(path "/f185fde3-43b8-46c7-bad3-2f317c19deaa"
 					(reference "U1")
 					(unit 1)
@@
 		(instances
 			(project "Inverting Amplifier"
-				(path "/08241a88-1f4f-4518-809a-7c34a0316343"
+				(path "/f185fde3-43b8-46c7-bad3-2f317c19deaa"
 					(reference "R1")
 					(unit 1)
@@
 		(instances
 			(project "Inverting Amplifier"
-				(path "/08241a88-1f4f-4518-809a-7c34a0316343"
+				(path "/f185fde3-43b8-46c7-bad3-2f317c19deaa"
 					(reference "R2")
 					(unit 1)
@@
 		(instances
 			(project "Inverting Amplifier"
-				(path "/08241a88-1f4f-4518-809a-7c34a0316343"
+				(path "/f185fde3-43b8-46c7-bad3-2f317c19deaa"
 					(reference "C1")
 					(unit 1)
@@
 		(instances
 			(project "Inverting Amplifier"
-				(path "/08241a88-1f4f-4518-809a-7c34a0316343"
+				(path "/f185fde3-43b8-46c7-bad3-2f317c19deaa"
 					(reference "C2")
 					(unit 1)
@@
 		(instances
 			(project "Inverting Amplifier"
-				(path "/08241a88-1f4f-4518-809a-7c34a0316343"
+				(path "/f185fde3-43b8-46c7-bad3-2f317c19deaa"
 					(reference "R3")
 					(unit 1)
@@
 		(instances
 			(project "Inverting Amplifier"
-				(path "/08241a88-1f4f-4518-809a-7c34a0316343"
+				(path "/f185fde3-43b8-46c7-bad3-2f317c19deaa"
 					(reference "#PWR01")
 					(unit 1)
@@
 		(instances
 			(project "Inverting Amplifier"
-				(path "/08241a88-1f4f-4518-809a-7c34a0316343"
+				(path "/f185fde3-43b8-46c7-bad3-2f317c19deaa"
 					(reference "#PWR02")
 					(unit 1)
@@
 		(instances
 			(project "Inverting Amplifier"
-				(path "/08241a88-1f4f-4518-809a-7c34a0316343"
+				(path "/f185fde3-43b8-46c7-bad3-2f317c19deaa"
 					(reference "#PWR03")
 					(unit 1)
@@
 		(instances
 			(project "Inverting Amplifier"
-				(path "/08241a88-1f4f-4518-809a-7c34a0316343"
+				(path "/f185fde3-43b8-46c7-bad3-2f317c19deaa"
 					(reference "#PWR04")
 					(unit 1)
@@
 		(instances
 			(project "Inverting Amplifier"
-				(path "/08241a88-1f4f-4518-809a-7c34a0316343"
+				(path "/f185fde3-43b8-46c7-bad3-2f317c19deaa"
 					(reference "V1")
 					(unit 1)
@@
 		(instances
 			(project "Inverting Amplifier"
-				(path "/08241a88-1f4f-4518-809a-7c34a0316343"
+				(path "/f185fde3-43b8-46c7-bad3-2f317c19deaa"
 					(reference "#PWR05")
 					(unit 1)
