File: sim_work/usb_ina.kicad_sch (KiCad schematic)
At the start: 14 parts, among them U1 LM741, U2 LM741, U3 LM741

Commit message: Add comparison mode, fix SimGUI subprocess popups, DAC7800 IC boxes
- SimGUI: fix Python path detection (FindPython searches Python312/313/311)
- SimGUI: suppress console popup windows (CREATE_NO_WINDOW for subprocess)
- SimGUI: add Comparison project (MDAC vs Analog oscillator side-by-side)
- SimGUI: fix async wrapping (direct await instead of Task.Run)
- Pipeline: draw DAC7800 as proper IC box with pin labels (VREF/IOUT/VCTRL)
- Pipeline: fix electrometer_362 layout (spacing, junction dots at T-junctions)
- Pipeline: fix summing amp gain annotations (BP=-0.455, not -2.2)
- Pipeline: add analog_osc command for friend's SVF oscillator simulation
- Docs: comparison_guide.md, updated README and PROJECT tracker

Co-Authored-By: Claude Opus 4.6 <noreply@anthropic.com>
Connections:
- net +12V: now also U1.4 (V-), U2.4 (V-), U3.4 (V-); no longer U1.7 (V+), U2.7 (V+), U3.7 (V+)
- net -12V: now also U1.7 (V+), U2.7 (V+), U3.7 (V+); no longer U1.4 (V-), U2.4 (V-), U3.4 (V-)
- net at R4.2, R6.1: now also U3.3 (+); no longer U3.2 (-)
- net at R1.1, R3.1: now also U1.3 (+); no longer U1.2 (-)
- net at R2.1, R3.2: now also U2.3 (+); no longer U2.2 (-)
- net at R5.2, R7.1: now also U3.2 (-); no longer U3.3 (+)
- net at V1.1: now also U1.2 (-); no longer U1.3 (+)
- net at V2.1: now also U2.2 (-); no longer U2.3 (+)
Changed lines of the file:
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@@
 		(lib_id "LM741:LM741")
 		(at 116.84 71.12 0)
-		(mirror x)
 		(unit 1)
 		(exclude_from_sim no)
@@
 		(instances
 			(project "Instrumentation Amplifier"
-				(path "/cb4aa8cf-b73c-41da-b5d3-1e4fee31bbc3"
+				(path "/d2fa4ebb-45af-4c56-afa0-acca04458505"
 					(reference "U1")
 					(unit 1)
@@
 		(lib_id "LM741:LM741")
 		(at 116.84 132.08 0)
-		(mirror x)
 		(unit 1)
 		(exclude_from_sim no)
@@
 		(instances
 			(project "Instrumentation Amplifier"
-				(path "/cb4aa8cf-b73c-41da-b5d3-1e4fee31bbc3"
+				(path "/d2fa4ebb-45af-4c56-afa0-acca04458505"
 					(reference "U2")
 					(unit 1)
@@
 		(lib_id "LM741:LM741")
 		(at 198.12 101.6 0)
-		(mirror x)
 		(unit 1)
 		(exclude_from_sim no)
@@
 		(instances
 			(project "Instrumentation Amplifier"
-				(path "/cb4aa8cf-b73c-41da-b5d3-1e4fee31bbc3"
+				(path "/d2fa4ebb-45af-4c56-afa0-acca04458505"
 					(reference "U3")
 					(unit 1)
@@
 		(instances
 			(project "Instrumentation Amplifier"
-				(path "/cb4aa8cf-b73c-41da-b5d3-1e4fee31bbc3"
+				(path "/d2fa4ebb-45af-4c56-afa0-acca04458505"
 					(reference "R1")
 					(unit 1)
@@
 		(instances
 			(project "Instrumentation Amplifier"
-				(path "/cb4aa8cf-b73c-41da-b5d3-1e4fee31bbc3"
+				(path "/d2fa4ebb-45af-4c56-afa0-acca04458505"
 					(reference "R2")
 					(unit 1)
@@
 		(instances
 			(project "Instrumentation Amplifier"
-				(path "/cb4aa8cf-b73c-41da-b5d3-1e4fee31bbc3"
+				(path "/d2fa4ebb-45af-4c56-afa0-acca04458505"
 					(reference "R3")
 					(unit 1)
@@
 		(instances
 			(project "Instrumentation Amplifier"
-				(path "/cb4aa8cf-b73c-41da-b5d3-1e4fee31bbc3"
+				(path "/d2fa4ebb-45af-4c56-afa0-acca04458505"
 					(reference "R4")
 					(unit 1)
@@
 		(instances
 			(project "Instrumentation Amplifier"
-				(path "/cb4aa8cf-b73c-41da-b5d3-1e4fee31bbc3"
+				(path "/d2fa4ebb-45af-4c56-afa0-acca04458505"
 					(reference "R5")
 					(unit 1)
@@
 		(instances
 			(project "Instrumentation Amplifier"
-				(path "/cb4aa8cf-b73c-41da-b5d3-1e4fee31bbc3"
+				(path "/d2fa4ebb-45af-4c56-afa0-acca04458505"
 					(reference "R6")
 					(unit 1)
@@
 		(instances
 			(project "Instrumentation Amplifier"
-				(path "/cb4aa8cf-b73c-41da-b5d3-1e4fee31bbc3"
+				(path "/d2fa4ebb-45af-4c56-afa0-acca04458505"
 					(reference "R7")
 					(unit 1)
@@
 		(instances
 			(project "Instrumentation Amplifier"
-				(path "/cb4aa8cf-b73c-41da-b5d3-1e4fee31bbc3"
+				(path "/d2fa4ebb-45af-4c56-afa0-acca04458505"
 					(reference "C1")
 					(unit 1)
@@
 		(instances
 			(project "Instrumentation Amplifier"
-				(path "/cb4aa8cf-b73c-41da-b5d3-1e4fee31bbc3"
+				(path "/d2fa4ebb-45af-4c56-afa0-acca04458505"
 					(reference "R8")
 					(unit 1)
@@
 		(instances
 			(project "Instrumentation Amplifier"
-				(path "/cb4aa8cf-b73c-41da-b5d3-1e4fee31bbc3"
+				(path "/d2fa4ebb-45af-4c56-afa0-acca04458505"
 					(reference "#PWR01")
 					(unit 1)
@@
 		(instances
 			(project "Instrumentation Amplifier"
-				(path "/cb4aa8cf-b73c-41da-b5d3-1e4fee31bbc3"
+				(path "/d2fa4ebb-45af-4c56-afa0-acca04458505"
 					(reference "#PWR02")
 					(unit 1)
@@
 		(instances
 			(project "Instrumentation Amplifier"
-				(path "/cb4aa8cf-b73c-41da-b5d3-1e4fee31bbc3"
+				(path "/d2fa4ebb-45af-4c56-afa0-acca04458505"
 					(reference "#PWR03")
 					(unit 1)
@@
 		(instances
 			(project "Instrumentation Amplifier"
-				(path "/cb4aa8cf-b73c-41da-b5d3-1e4fee31bbc3"
+				(path "/d2fa4ebb-45af-4c56-afa0-acca04458505"
 					(reference "#PWR04")
 					(unit 1)
@@
 		(instances
 			(project "Instrumentation Amplifier"
-				(path "/cb4aa8cf-b73c-41da-b5d3-1e4fee31bbc3"
+				(path "/d2fa4ebb-45af-4c56-afa0-acca04458505"
 					(reference "#PWR05")
 					(unit 1)
@@
 		(instances
 			(project "Instrumentation Amplifier"
-				(path "/cb4aa8cf-b73c-41da-b5d3-1e4fee31bbc3"
+				(path "/d2fa4ebb-45af-4c56-afa0-acca04458505"
 					(reference "#PWR06")
 					(unit 1)
@@
 		(instances
 			(project "Instrumentation Amplifier"
-				(path "/cb4aa8cf-b73c-41da-b5d3-1e4fee31bbc3"
+				(path "/d2fa4ebb-45af-4c56-afa0-acca04458505"
 					(reference "#PWR07")
 					(unit 1)
@@
 		(instances
 			(project "Instrumentation Amplifier"
-				(path "/cb4aa8cf-b73c-41da-b5d3-1e4fee31bbc3"
+				(path "/d2fa4ebb-45af-4c56-afa0-acca04458505"
 					(reference "#PWR08")
 					(unit 1)
@@
 		(instances
 			(project "Instrumentation Amplifier"
-				(path "/cb4aa8cf-b73c-41da-b5d3-1e4fee31bbc3"
+				(path "/d2fa4ebb-45af-4c56-afa0-acca04458505"
 					(reference "V1")
 					(unit 1)
@@
 		(instances
 			(project "Instrumentation Amplifier"
-				(path "/cb4aa8cf-b73c-41da-b5d3-1e4fee31bbc3"
+				(path "/d2fa4ebb-45af-4c56-afa0-acca04458505"
 					(reference "#PWR09")
 					(unit 1)
@@
 		(instances
 			(project "Instrumentation Amplifier"
-				(path "/cb4aa8cf-b73c-41da-b5d3-1e4fee31bbc3"
+				(path "/d2fa4ebb-45af-4c56-afa0-acca04458505"
 					(reference "V2")
 					(unit 1)
@@
 		(instances
 			(project "Instrumentation Amplifier"
-				(path "/cb4aa8cf-b73c-41da-b5d3-1e4fee31bbc3"
+				(path "/d2fa4ebb-45af-4c56-afa0-acca04458505"
 					(reference "#PWR10")
 					(unit 1)
